File: elec/layout/default/logic-card.kicad_pcb (KiCad board)
At the start: 2 copper layers, 76 x 68 mm, 53 parts

Commit message: add new layout
Parts:
- R10, R11: value 10.0 KΩ -> Chip Resistor - Surface Mount 11KOhms ±5% 1/16W 0402 RoHS; footprint lib:C0603 -> lib:R0402
- R12, R13, R14, R15, R16, R2, R6, R7: value 10.0 KΩ -> Chip Resistor - Surface Mount 10KOhms ±5% 1/16W 0402 RoHS
- R17: value 1.5 KΩ -> Chip Resistor - Surface Mount 1.5KOhms ±5% 1/10W 0603 RoHS
- R18, R19: value 100.0 Ω -> Chip Resistor - Surface Mount 100Ohms ±5% 1/10W 0603 RoHS
- R3: value 1.0 KΩ -> Chip Resistor - Surface Mount 1KOhms ±5% 1/16W 0402 RoHS
Connections:
- C3 pad 1: xin -> vcc-4
- C4 pad 1: out-1 -> vcc-5
- R1 pad 2: adj -> io
- R2 pad 1: adj -> io
- R3 pad 2: out-1 -> vcc-5
- U12 pad A4: vcc-4 -> vcc-6
- U12 pad A9: vcc-4 -> vcc-6
- U12 pad B4: vcc-4 -> vcc-6
- U12 pad B9: vcc-4 -> vcc-6
- U13 pad 2: vcc-4 -> vcc-6
- U16 pad 8: out-2 -> out-1
- U7 pad 20: xin -> vcc-4
- U8 pad 1: xin -> vcc-4
- U8 pad 3: out-1 -> vcc-5
Routing:
- net vcc-6: track 0.00 -> 11.3 mm
- net xin: track 9.03 -> 0.00 mm
- net io: track 0.00 -> 6.43 mm
- net adj: track 6.43 -> 0.00 mm
- net vcc-5: track 0.00 -> 3.09 mm
- net vcc-4: track 11.3 -> 9.03 mm
